File: Allwinner_V3S/Allwinner_V3S/Allwinner_V3S.kicad_pcb (KiCad board)
At the start: 2 copper layers, 47 parts, among them U1 Allwinner_V3S, U2 SY8088AAC, U3 SY8088AAC, U4 SY8088AAC, U5 CH340N, U6 XC6206PxxxMR, U7 FPC_24, Y1 32.768K, Y2 24M

Commit message: update
Parts:
- removed R13, R14, R15: 10K, Resistor_SMD:R_0402_1005Metric
- removed U7: FPC_24, mypack:Hirose_FH12-24S-0.5SH_1x24-1MP_P0.50mm_Horizontal
- added C17: 104, Capacitor_SMD:C_0402_1005Metric, F.Cu at (161.7, 74.5)
- added C18: 104, Capacitor_SMD:C_0402_1005Metric, F.Cu at (158.8, 74.5)
- added C19: 104, Capacitor_SMD:C_0402_1005Metric, F.Cu at (155.9, 76.4)
- added R19: 0/NC, Resistor_SMD:R_0402_1005Metric, F.Cu at (172.2, 65.5)
- added R20: 0/NC, Resistor_SMD:R_0402_1005Metric, F.Cu at (153.0, 74.5)
- added U9: OV7724_FPC_24PIN, mypack:Hirose_FH12-24S-0.5SH_1x24-1MP_P0.50mm_Horizontal, F.Cu at (161.2, 68.0)
- C2: value C_0402 -> 104
- R2: value R_0402 -> 10K
- moved U2 24.8 mm to (114.9, 81.4)
- moved C2 24.6 mm to (172.2, 67.5)
- moved L2 21.5 mm to (142.2, 65.9)
- moved C6 17.8 mm to (147.1, 69.5)
- moved R3 17.5 mm to (132.6, 81.2)
- moved U6 17.2 mm to (133.7, 77.9)
- moved C7 17.1 mm to (137.3, 78.6)
- moved U4 16.6 mm to (133.9, 73.3)
- moved R11 16.0 mm to (137.3, 76.6)
- moved L3 14.1 mm to (124.4, 80.5)
- moved R2 13.8 mm to (156.0, 74.5)
- moved C16 13.7 mm to (117.3, 73.5)
- moved R1 13.2 mm to (153.0, 76.5)
- moved C9 13.1 mm to (134.0, 83.1)
- moved R10 11.6 mm to (137.7, 74.0)
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Connections:
- C2 pad 1: Net-(C2-Pad1) -> +3V3
- C2 pad 2: Net-(C2-Pad2) -> GND
- R1 pad 1: Net-(R1-Pad1) -> /camera/OV7725_RESET
- R1 pad 2: +2V8 -> +3V3
- R2 pad 1: Net-(R2-Pad1) -> GND
- R2 pad 2: Net-(R2-Pad2) -> /camera/OV7725_PWDN
- U1 pad 16: /camera_fpc24/PE15_CSI_D11_LCD_D15 -> /camera/OV7725_Y9
- U1 pad 17: /camera_fpc24/PE14_CSI_D10_LCD_D14 -> /camera/OV7725_Y8
- U1 pad 18: /camera_fpc24/PE13_CSI_D9_LCD_D13 -> /camera/OV7725_Y7
- U1 pad 22: /camera_fpc24/PE12_CSI_D8_LCD_D12 -> /camera/OV7725_Y6
- U1 pad 23: /camera_fpc24/PE11_CSI_D7_LCD_D11 -> /camera/OV7725_Y5
- U1 pad 24: /camera_fpc24/PE10_CSI_D7_LCD_D10 -> /camera/OV7725_Y4
- U1 pad 27: /camera_fpc24/PE9_CSI_D5_LCD7 -> /camera/OV7725_Y3
- U1 pad 28: /camera_fpc24/PE8_CSI_D4_LCD_D6 -> /camera/OV7725_Y2
- U1 pad 34: /camera_fpc24/PE3_CSI_VSYNCLCD_VSYNC -> /camera/OV7725_VSYNC
- U1 pad 35: /camera_fpc24/PE2_CSI_HSYSNC_LCD_HSYNC -> /camera/OV7725_HREF
- U1 pad 36: /camera_fpc24/PE1_CSI_MCLK_LCD_DE -> /camera/OV7725_MCLK
- U1 pad 37: /camera_fpc24/PE0_CSI_PCLK_LCD_CLK -> /camera/OV7725_PCLK
- U1 pad 8: /camera_fpc24/PE22_CSI_SDA_TWI1_SDA_UART1_RX -> /camera/OV7725_SIO-D
- U1 pad 9: /camera_fpc24/PE21_CSI_SCK_TWI1_SCK_UART1_TX -> /camera/OV7725_SIO-C
