File: Allwinner_V3S/Allwinner_V3S/Allwinner_V3S.sch (KiCad schematic (older format))
At the start: 2 parts

Commit message: update
Parts:
- removed C2: C_0402, Capacitor_SMD:C_0402_1005Metric, symbol mylib:C_0402
- removed R2: R_0402, Resistor_SMD:R_0402_1005Metric, symbol mylib:R_0402
Connections:
- no-connect marks 0 -> 2
Changed lines of the file:
@@
 $Descr A2 23386 16535
 encoding utf-8
-Sheet 1 6
+Sheet 1 4
 Title ""
 Date ""
@@
 F10 "USB1_DN" I R 5450 6100 50
 $EndSheet
-$Comp
-L mylib:C_0402 C2
-U 1 1 62465CD5
-P 4275 3400
-F 0 "C2" H 3925 3400 50  0000 L CNN
-F 1 "C_0402" H 3875 3300 50  0000 L CNN
-F 2 "Capacitor_SMD:C_0402_1005Metric" V 4125 3300 50  0001 C CNN
-F 3 "" V 4125 3300 50  0001 C CNN
-	1    4275 3400
-	1    0    0    -1
-$EndComp
-$Comp
-L mylib:R_0402 R2
-U 1 1 6245BA0C
-P 3775 3000
-F 0 "R2" H 3845 3046 50  0000 L CNN
-F 1 "R_0402" H 3845 2955 50  0000 L CNN
-F 2 "Resistor_SMD:R_0402_1005Metric" H 4075 2750 50  0001 C CNN
-F 3 "" H 3475 3150 50  0001 C CNN
-	1    3775 3000
-	1    0    0    -1
-$EndComp
 $Comp
 L power:+1V8 #PWR035
@@
 	0    1    1    0
 $EndComp
-$Sheet
-S 4100 8125 1450 2300
-U 624CABEC
-F0 "camera_fpc24" 50
-F1 "camera_fpc24.sch" 50
-F2 "PE2_CSI_HSYSNC_LCD_HSYNC" I R 5550 10075 50
-F3 "PE0_CSI_PCLK_LCD_CLK" I R 5550 10275 50
-F4 "PE1_CSI_MCLK_LCD_DE" I R 5550 10175 50
-F5 "PE22_CSI_SDA_TWI1_SDA_UART1_RX" I R 5550 8550 50
-F6 "PE21_CSI_SCK_TWI1_SCK_UART1_TX" I R 5550 8650 50
-F7 "PE8_CSI_D4_LCD_D6" I R 5550 9650 50
-F8 "PE9_CSI_D5_LCD7" I R 5550 9550 50
-F9 "PE10_CSI_D7_LCD_D10" I R 5550 9450 50
-F10 "PE11_CSI_D7_LCD_D11" I R 5550 9350 50
-F11 "PE12_CSI_D8_LCD_D12" I R 5550 9250 50
-F12 "PE13_CSI_D9_LCD_D13" I R 5550 9150 50
-F13 "PE14_CSI_D10_LCD_D14" I R 5550 9050 50
-F14 "PE15_CSI_D11_LCD_D15" I R 5550 8950 50
-F15 "PE3_CSI_VSYNCLCD_VSYNC" I R 5550 9975 50
-$EndSheet
 $Sheet
 S 6375 4875 3500 5550
@@
 	5450 5750 6375 5750
 $Sheet
-S 15225 5075 2100 2375
-U 624953A8
-F0 "display" 50
-F1 "display.sch" 50
-$EndSheet
-$Sheet
-S 11450 5900 1050 2125
+S 4450 8375 1100 2025
 U 624985F7
 F0 "camera" 50
 F1 "camera.sch" 50
+F2 "OV7725_SIO-D" I R 5550 8550 50
+F3 "OV7725_SIO-C" I R 5550 8650 50
+F4 "OV7725_RESET" I R 5550 8750 50
+F5 "OV7725_VSYNC" I R 5550 9975 50
+F6 "OV7725_PWDN" I R 5550 8850 50
+F7 "OV7725_HREF" I R 5550 10075 50
+F8 "OV7725_MCLK" I R 5550 10175 50
+F9 "OV7725_Y8" I R 5550 9050 50
+F10 "OV7725_Y7" I R 5550 9150 50
+F11 "OV7725_PCLK" I R 5550 10275 50
+F12 "OV7725_Y6" I R 5550 9250 50
+F13 "OV7725_Y2" I R 5550 9650 50
+F14 "OV7725_Y5" I R 5550 9350 50
+F15 "OV7725_Y3" I R 5550 9550 50
+F16 "OV7725_Y4" I R 5550 9450 50
+F17 "OV7725_Y9" I R 5550 8950 50
 $EndSheet
+NoConn ~ 5550 8850
+NoConn ~ 5550 8750
 $EndSCHEMATC
