File: Allwinner_V3S/Allwinner_V3S/camera.sch (KiCad schematic (older format))
At the start: 6 parts, among them U9 OV7724_FPC_24PIN

Commit message: update
Parts:
- added C2: 104, Capacitor_SMD:C_0402_1005Metric, symbol mylib:C_0402
- added R1, R2: 10K, Resistor_SMD:R_0402_1005Metric, symbol mylib:R_0402
Connections:
- net labels added: OV7725_Y9
- net labels removed: OV7725_Y0, OV7725_Y1
- wire segments 34 -> 35
Other:
- moved on the sheet: C17, C18
Changed lines of the file:
@@
 $Descr A4 11693 8268
 encoding utf-8
-Sheet 6 6
+Sheet 4 4
 Title ""
 Date ""
@@
 L mylib:C_0402 C18
 U 1 1 624A1195
-P 3850 2375
-F 0 "C18" H 3965 2421 50  0000 L CNN
-F 1 "104" H 3965 2330 50  0000 L CNN
-F 2 "Capacitor_SMD:C_0402_1005Metric" V 3700 2275 50  0001 C CNN
-F 3 "" V 3700 2275 50  0001 C CNN
-	1    3850 2375
+P 2125 2375
+F 0 "C18" H 2240 2421 50  0000 L CNN
+F 1 "104" H 2240 2330 50  0000 L CNN
+F 2 "Capacitor_SMD:C_0402_1005Metric" V 1975 2275 50  0001 C CNN
+F 3 "" V 1975 2275 50  0001 C CNN
+	1    2125 2375
 	1    0    0    -1
 $EndComp
@@
 Text HLabel 5175 4000 0    50   Input ~ 0
 OV7725_Y4
-Text HLabel 5175 4100 0    50   Input ~ 0
-OV7725_Y1
-Text HLabel 5175 4200 0    50   Input ~ 0
-OV7725_Y0
 Wire Wire Line
 	5175 3400 5425 3400
@@
 Wire Wire Line
 	5175 4000 5425 4000
-Wire Wire Line
-	5175 4100 5425 4100
-Wire Wire Line
-	5175 4200 5425 4200
 Wire Wire Line
 	5175 3200 5425 3200
@@
 	5175 3100 5425 3100
 Text HLabel 5175 3000 0    50   Input ~ 0
-OV7725_Y8
+OV7725_Y9
 Wire Wire Line
 	5175 3000 5425 3000
@@
 L power:+3.3V #PWR075
 U 1 1 624ABDDC
-P 3850 2225
-F 0 "#PWR075" H 3850 2075 50  0001 C CNN
-F 1 "+3.3V" H 3865 2398 50  0000 C CNN
-F 2 "" H 3850 2225 50  0001 C CNN
-F 3 "" H 3850 2225 50  0001 C CNN
-	1    3850 2225
+P 2125 2225
+F 0 "#PWR075" H 2125 2075 50  0001 C CNN
+F 1 "+3.3V" H 2140 2398 50  0000 C CNN
+F 2 "" H 2125 2225 50  0001 C CNN
+F 3 "" H 2125 2225 50  0001 C CNN
+	1    2125 2225
 	1    0    0    -1
 $EndComp
@@
 L power:GND #PWR074
 U 1 1 624AC6BC
-P 3700 2525
-F 0 "#PWR074" H 3700 2275 50  0001 C CNN
-F 1 "GND" H 3705 2352 50  0000 C CNN
-F 2 "" H 3700 2525 50  0001 C CNN
-F 3 "" H 3700 2525 50  0001 C CNN
-	1    3700 2525
+P 1975 2525
+F 0 "#PWR074" H 1975 2275 50  0001 C CNN
+F 1 "GND" H 1980 2352 50  0000 C CNN
+F 2 "" H 1975 2525 50  0001 C CNN
+F 3 "" H 1975 2525 50  0001 C CNN
+	1    1975 2525
 	1    0    0    -1
 $EndComp
@@
 L power:+1V8 #PWR073
 U 1 1 624AD4E4
-P 3550 2225
-F 0 "#PWR073" H 3550 2075 50  0001 C CNN
-F 1 "+1V8" H 3565 2398 50  0000 C CNN
-F 2 "" H 3550 2225 50  0001 C CNN
-F 3 "" H 3550 2225 50  0001 C CNN
-	1    3550 2225
+P 1825 2225
+F 0 "#PWR073" H 1825 2075 50  0001 C CNN
+F 1 "+1V8" H 1840 2398 50  0000 C CNN
+F 2 "" H 1825 2225 50  0001 C CNN
+F 3 "" H 1825 2225 50  0001 C CNN
+	1    1825 2225
 	1    0    0    -1
 $EndComp
@@
 L mylib:C_0402 C17
 U 1 1 624ADFE3
-P 3550 2375
-F 0 "C17" H 3665 2421 50  0000 L CNN
-F 1 "104" H 3665 2330 50  0000 L CNN
-F 2 "Capacitor_SMD:C_0402_1005Metric" V 3400 2275 50  0001 C CNN
-F 3 "" V 3400 2275 50  0001 C CNN
-	1    3550 2375
-	1    0    0    -1
-$EndComp
-Wire Wire Line
-	3550 2525 3700 2525
-Connection ~ 3700 2525
-Wire Wire Line
-	3700 2525 3850 2525
+P 1825 2375
+F 0 "C17" H 1940 2421 50  0000 L CNN
+F 1 "104" H 1940 2330 50  0000 L CNN
+F 2 "Capacitor_SMD:C_0402_1005Metric" V 1675 2275 50  0001 C CNN
+F 3 "" V 1675 2275 50  0001 C CNN
+	1    1825 2375
+	1    0    0    -1
+$EndComp
+Wire Wire Line
+	1825 2525 1975 2525
+Connection ~ 1975 2525
+Wire Wire Line
+	1975 2525 2125 2525
 Wire Wire Line
 	4500 2900 4650 2900
@@
 Wire Wire Line
 	4150 3000 4200 3000
+$Comp
+L power:+3.3V #PWR027
+U 1 1 624C9E33
+P 5150 4200
+F 0 "#PWR027" H 5150 4050 50  0001 C CNN
+F 1 "+3.3V" V 5165 4328 50  0000 L CNN
+F 2 "" H 5150 4200 50  0001 C CNN
+F 3 "" H 5150 4200 50  0001 C CNN
+	1    5150 4200
+	-1   0    0    1
+$EndComp
+$Comp
+L power:GND #PWR03
+U 1 1 624CAA48
+P 4850 4100
+F 0 "#PWR03" H 4850 3850 50  0001 C CNN
+F 1 "GND" V 4855 3972 50  0000 R CNN
+F 2 "" H 4850 4100 50  0001 C CNN
+F 3 "" H 4850 4100 50  0001 C CNN
+	1    4850 4100
+	0    1    1    0
+$EndComp
+Wire Wire Line
+	5150 4200 5425 4200
+$Comp
+L mylib:C_0402 C2
+U 1 1 624CE78C
+P 5000 4200
+F 0 "C2" H 5115 4246 50  0000 L CNN
+F 1 "104" H 5115 4155 50  0000 L CNN
+F 2 "Capacitor_SMD:C_0402_1005Metric" V 4850 4100 50  0001 C CNN
+F 3 "" V 4850 4100 50  0001 C CNN
+	1    5000 4200
+	0    1    1    0
+$EndComp
+Connection ~ 5150 4200
+Wire Wire Line
+	4850 4100 5425 4100
+Wire Wire Line
+	4850 4200 4850 4100
+Connection ~ 4850 4100
+Text HLabel 3225 2350 0    50   Input ~ 0
+OV7725_RESET
+$Comp
+L mylib:R_0402 R1
+U 1 1 624D334F
+P 3225 2200
+F 0 "R1" V 3125 2150 50  0000 C CNN
+F 1 "10K" V 3225 2200 50  0000 C CNN
+F 2 "Resistor_SMD:R_0402_1005Metric" H 3525 1950 50  0001 C CNN
+F 3 "" H 2925 2350 50  0001 C CNN
+	1    3225 2200
+	-1   0    0    1
+$EndComp
+$Comp
+L power:+3.3V #PWR01
+U 1 1 624D3B3C
+P 3225 2050
+F 0 "#PWR01" H 3225 1900 50  0001 C CNN
+F 1 "+3.3V" H 3240 2223 50  0000 C CNN
+F 2 "" H 3225 2050 50  0001 C CNN
+F 3 "" H 3225 2050 50  0001 C CNN
+	1    3225 2050
+	1    0    0    -1
+$EndComp
+Text HLabel 3225 2500 0    50   Input ~ 0
+OV7725_PWDN
+$Comp
+L mylib:R_0402 R2
+U 1 1 624DFC51
+P 3225 2650
+F 0 "R2" V 3125 2600 50  0000 C CNN
+F 1 "10K" V 3225 2650 50  0000 C CNN
+F 2 "Resistor_SMD:R_0402_1005Metric" H 3525 2400 50  0001 C CNN
+F 3 "" H 2925 2800 50  0001 C CNN
+	1    3225 2650
+	-1   0    0    1
+$EndComp
+$Comp
+L power:GND #PWR02
+U 1 1 624E0140
+P 3225 2800
+F 0 "#PWR02" H 3225 2550 50  0001 C CNN
+F 1 "GND" V 3230 2672 50  0000 R CNN
+F 2 "" H 3225 2800 50  0001 C CNN
+F 3 "" H 3225 2800 50  0001 C CNN
+	1    3225 2800
+	1    0    0    -1
+$EndComp
 $EndSCHEMATC
